File: Project/MCU-DB-STM32H750VB-FULL/MCU-DB-STM32H750VB-FULL.kicad_sch (KiCad schematic)
At the start: 5 parts, among them J1 NPPN402AFCN-RC, J2 NPPN402AFCN-RC, J3 FTSH-107-01-L-DV-K, U1 STM32H750VBTx, U2 AMS1117-3.3

Commit message: Schematic updated
Parts:
- added C1, C2: 20pF, 22L_CAPACITOR_SMD:C0805_Long_Pad, symbol 22L_CAPACITOR_SMD:20pF
- added C10, C11, C12, C13, C14, C15, C16, C17, C18, C20, C22, C24, C27, C28, C29, C3, C33, C4, C5, C6, C7, C8, C9: 100nF, 22L_CAPACITOR_SMD:C0805_Long_Pad, symbol 22L_CAPACITOR_SMD:104
- added C19, C32: 1uF, 22L_CAPACITOR_SMD:C0805_Long_Pad, symbol 22L_CAPACITOR_SMD:1μF
- added C21, C23, C26: 10μF, 22L_CAPACITOR_SMD:C0805_Long_Pad, symbol 22L_CAPACITOR_SMD:10μF
- added C25: 10nF, 22L_CAPACITOR_SMD:C0805_Long_Pad, symbol 22L_CAPACITOR_SMD:103
- added C30, C31: 2.2μF, 22L_CAPACITOR_SMD:C0805_Long_Pad, symbol 22L_CAPACITOR_SMD:2.2μF
- added J4: 10118192-0002LF, 22L_USB_CONNECTOR:AMPHENOL_10118192-0002LF, symbol 22L_USB_CONNECTOR:10118192-0002LF
- added JP1: SolderJumper_2_Open, Jumper:SolderJumper-2_P1.3mm_Open_RoundedPad1.0x1.5mm, symbol Jumper:SolderJumper_2_Open
- added LED1, LED2: SZYY0805YG, 22L_LED_SMD:LED0805-R-RD_GREEN, symbol 22L_LED_SMD:SZYY0805YG_1
- added R1, R6, R7: 10K, 22L_RESISTOR_SMD:R0805_Long_Pad, symbol 22L_RESISTOR_SMD:10K
- added R10, R11, R5: 330R, 22L_RESISTOR_SMD:R0805_Long_Pad, symbol 22L_RESISTOR_SMD:330R
- added R2: 10M, 22L_RESISTOR_SMD:R0805_Long_Pad, symbol 22L_RESISTOR_SMD:10M
- added R3, R4: 0R, 22L_RESISTOR_SMD:R0805_Long_Pad, symbol 22L_RESISTOR_SMD:0R
- added R8, R9: 22R, 22L_RESISTOR_SMD:R0805_Long_Pad, symbol 22L_RESISTOR_SMD:22R
- added S1: JS202011SCQN, 22L_SWITCH_SMD:SW_JS202011SCQN, symbol 22L_SWITCH_SMD:JS202011SCQN
- added SW1: SW_Push_Dual, 22L_SWITCH_SMD:SMT_MTRLFS_CNK, symbol 22L_SWITCH_SMD:SW_Push_Dual
- added U3: STMPS2151STR, SOT23-5L_STM, symbol 22L_LOAD_DRIVERS:STMPS2151STR
- added Y1: ECS-80-20-20A-TR, ECS-80-20-20A-TR:XTAL_ECS-80-20-20A-TR, symbol 22L_CRYSTAL_SMD:ECS-80-20-20A-TR
- J1, J2: Digikey part number (none) -> S5801-40-ND
Connections:
- net VREF+ is gone; now on net +3.3V: J1.34 (VREF+)
- net BOOT0: now also R1.1
- net GND: now also U2.1 (GND), C1.2, C10.2, C11.2, C12.2, C13.2, C14.2, C15.2, C16.2, C17.2, C18.2, C19.2, C2.2, C20.2, C21.2, C22.2, C23.2, C24.2, C25.1, C26.2, C27.2, C28.2, C29.2, C3.2, C30.2, C31.2, C32.2, C33.2, C4.2, C5.2, C6.2, C7.2, C8.2, C9.2, J4.5 (GND), J4.S1 (SHIELD), J4.S2 (SHIELD__1), J4.S3 (SHIELD__2), J4.S4 (SHIELD__3), J4.S5 (SHIELD__4), J4.S6 (SHIELD__5), LED1.1 (K), LED2.1 (K), R7.1, S1.3, SW1.1, SW1.3, U3.2 (GND)
- net PA10: now also R10.2
- net PH0: now also C1.1, R2.1, R4.2, Y1.1
- net PH1: now also C2.1, R2.2, R3.1, Y1.2
- net RESET: now also C25.2, SW1.2, SW1.4
- net VCAP_1: now reaches U1.48 (VCAP)
- net VCAP_1: now also C31.1
- net VCP_TX: now reaches U1.53 (PB14)
- net VCP_TX: now also J3.14 (VCP_TX)
- net VCP_RX: now reaches U1.54 (PB15)
- net VCP_RX: now also J3.13 (VCP_RX)
- net SWDIO: now reaches U1.72 (PA13)
- net SWDIO: now also J3.04 (SWDIO)
- net VCAP_2: now reaches U1.73 (VCAP)
- net VCAP_2: now also C30.1
- net SWCLK: now reaches U1.76 (PA14)
- net SWCLK: now also J3.06 (SWCLK)
- net +3.3V: now reaches U2.2 (VO)
- net +3.3V: now also C10.1, C11.1, C12.1, C13.1, C14.1, C15.1, C16.1, C17.1, C18.1, C23.1, C24.1, C3.1, C32.1, C33.1, C4.1, C5.1, C6.1, C7.1, C8.1, C9.1, R5.1, R6.2, S1.1
- net +5V: now reaches U2.3 (VI)
- net +5V: now also C21.1, C22.1, C29.1, U3.5 (IN)
- new net: J4.4 (ID), R10.1
- new net: LED2.2 (A), R11.2
- new net: R1.2, S1.2
- new net: LED1.2 (A), R5.2
- new net FLG: C27.1, R6.1, U3.3 (FAULT)
- new net OSC_IN: R4.1
- new net OSC_OUT: R3.2
- new net OTG_DM: R8.2
- new net OTG_DP: R9.2
- new net OTG_PWR_OUT: JP1.2 (B)
- new net USB 5V: C26.1, C28.1, J4.1 (VCC), R11.1, U3.1 (OUT)
- new net USBDM: J4.2 (D-), R8.1
- new net USBDP: J4.3 (D+), R9.1
- new net VBUSBEN: JP1.1 (A), R7.2, U3.4 (EN)
- new net VDDA: C19.1, C20.1
Other:
- moved on the sheet: J3, U2

Commit message: Schematic updated
Parts:
- removed R11: 330R, 22L_RESISTOR_SMD:R0805_Long_Pad, symbol 22L_RESISTOR_SMD:330R
- added R11: 1K, 22L_RESISTOR_SMD:R0805_Long_Pad, symbol 22L_RESISTOR_SMD:1K
Connections:
- net +3.3V: now also S1.4
- net GND: now also J3.05 (GND), J3.07 (GND), S1.6
- net USB 5V: now also R11.1
- net at LED2.2 (A): now also R11.2
- net at R1.2, S1.2: now also S1.5
Other:
- moved on the sheet: C32, C33, J3, J4, JP1, R1, R10, R8, R9
